Commit message: Get tesseract trajopt examples working

File: tesseract_ros/tesseract_examples/trajopt_examples/urdf/car_seat_demo.xacro (robot description, xacro)
@@ -1,5 +1,5 @@
 <?xml version="1.0" ?>
 <robot name="car_seat_demo" xmlns:xacro="http://ros.org/wiki/xacro">
-    <xacro:include filename="$(find motoman_sia20d_support)/urdf/sia20d_macro.xacro"/>
+    <xacro:include filename="$(find trajopt_examples)/urdf/sia20d_macro.xacro"/>
     <xacro:motoman_sia20d prefix=""/>
     <xacro:include filename="$(find trajopt_examples)/urdf/car_seat_demo_macro.xacro"/>

File: tesseract_ros/tesseract_examples/trajopt_examples/urdf/car_seat_demo_macro.xacro (robot description, xacro)
@@ -239,5 +239,68 @@
             <origin ryp="0 0 0" xyz="0 0 0"/>
             <geometry>
-              <mesh scale="0.9 0.9 0.9" filename="package://trajopt_examples/meshes/car_seat/collision/seat.stl"/>
+              <mesh scale="0.9 0.9 0.9" filename="package://trajopt_examples/meshes/car_seat/collision/seat_1.stl"/>
+            </geometry>
+            <material name="yellow"/>
+          </collision>
+          <collision>
+            <origin ryp="0 0 0" xyz="0 0 0"/>
+            <geometry>
+              <mesh scale="0.9 0.9 0.9" filename="package://trajopt_examples/meshes/car_seat/collision/seat_2.stl"/>
+            </geometry>
+            <material name="yellow"/>
+          </collision>
+          <collision>
+            <origin ryp="0 0 0" xyz="0 0 0"/>
+            <geometry>
+              <mesh scale="0.9 0.9 0.9" filename="package://trajopt_examples/meshes/car_seat/collision/seat_3.stl"/>
+            </geometry>
+            <material name="yellow"/>
+          </collision>
+          <collision>
+            <origin ryp="0 0 0" xyz="0 0 0"/>
+            <geometry>
+              <mesh scale="0.9 0.9 0.9" filename="package://trajopt_examples/meshes/car_seat/collision/seat_4.stl"/>
+            </geometry>
+            <material name="yellow"/>
+          </collision>
+          <collision>
+            <origin ryp="0 0 0" xyz="0 0 0"/>
+            <geometry>
+              <mesh scale="0.9 0.9 0.9" filename="package://trajopt_examples/meshes/car_seat/collision/seat_5.stl"/>
+            </geometry>
+            <material name="yellow"/>
+          </collision>
+          <collision>
+            <origin ryp="0 0 0" xyz="0 0 0"/>
+            <geometry>
+              <mesh scale="0.9 0.9 0.9" filename="package://trajopt_examples/meshes/car_seat/collision/seat_6.stl"/>
+            </geometry>
+            <material name="yellow"/>
+          </collision>
+          <collision>
+            <origin ryp="0 0 0" xyz="0 0 0"/>
+            <geometry>
+              <mesh scale="0.9 0.9 0.9" filename="package://trajopt_examples/meshes/car_seat/collision/seat_7.stl"/>
+            </geometry>
+            <material name="yellow"/>
+          </collision>
+          <collision>
+            <origin ryp="0 0 0" xyz="0 0 0"/>
+            <geometry>
+              <mesh scale="0.9 0.9 0.9" filename="package://trajopt_examples/meshes/car_seat/collision/seat_8.stl"/>
+            </geometry>
+            <material name="yellow"/>
+          </collision>
+          <collision>
+            <origin ryp="0 0 0" xyz="0 0 0"/>
+            <geometry>
+              <mesh scale="0.9 0.9 0.9" filename="package://trajopt_examples/meshes/car_seat/collision/seat_9.stl"/>
+            </geometry>
+            <material name="yellow"/>
+          </collision>
+          <collision>
+            <origin ryp="0 0 0" xyz="0 0 0"/>
+            <geometry>
+              <mesh scale="0.9 0.9 0.9" filename="package://trajopt_examples/meshes/car_seat/collision/seat_10.stl"/>
             </geometry>
             <material name="yellow"/>
@@ -304,5 +367,5 @@
           <child link="end_effector"/>
         </joint>
-        <!--<joint name="${prefix}end_effector_seat" type="fixed">
+<!--        <joint name="${prefix}end_effector_seat" type="fixed">
           <origin rpy="0 0.29 1.57" xyz="0.14 -0.1 -0.46"/>
           <parent link="end_effector"/>
