Commit message: Generate urdf files

File: tesseract_support/urdf/puzzle_piece_workcell.urdf (robot description, URDF)
Before this commit: robot puzzle_piece_workcell, 20 links, 19 joints
Links:
- link base_link: geometry collision mesh filename=package://tesseract_support/meshes/lbr_iiwa_14_r820/collisi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; visual mesh filename=package://tesseract_support/meshes/lbr_iiwa_14_r820/visual/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
- link ee_base: geometry collision mesh filename=package://tesseract_support/meshes/puzzle_piece/puzzle_moun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; visual mesh filename=package://tesseract_support/meshes/puzzle_piece/puzzle_moun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
- link grinder_base: geometry collision mesh filename=package://tesseract_support/meshes/puzzle_piece/grinder_col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; visual mesh filename=package://tesseract_support/meshes/puzzle_piece/grinder_vis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
- link link_1: geometry collision mesh filename=package://tesseract_support/meshes/lbr_iiwa_14_r820/collisi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; visual mesh filename=package://tesseract_support/meshes/lbr_iiwa_14_r820/visual/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
- link link_2: geometry collision mesh filename=package://tesseract_support/meshes/lbr_iiwa_14_r820/collisi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; visual mesh filename=package://tesseract_support/meshes/lbr_iiwa_14_r820/visual/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
- link link_3: geometry collision mesh filename=package://tesseract_support/meshes/lbr_iiwa_14_r820/collisi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; visual mesh filename=package://tesseract_support/meshes/lbr_iiwa_14_r820/visual/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
- link link_4: geometry collision mesh filename=package://tesseract_support/meshes/lbr_iiwa_14_r820/collisi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; visual mesh filename=package://tesseract_support/meshes/lbr_iiwa_14_r820/visual/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
- link link_5: geometry collision mesh filename=package://tesseract_support/meshes/lbr_iiwa_14_r820/collisi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; visual mesh filename=package://tesseract_support/meshes/lbr_iiwa_14_r820/visual/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
- link link_6: geometry collision mesh filename=package://tesseract_support/meshes/lbr_iiwa_14_r820/collisi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; visual mesh filename=package://tesseract_support/meshes/lbr_iiwa_14_r820/visual/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
- link link_7: geometry collision mesh filename=package://tesseract_support/meshes/lbr_iiwa_14_r820/collisi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; visual mesh filename=package://tesseract_support/meshes/lbr_iiwa_14_r820/visual/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
- link part: geometry collision mesh filename=package://tesseract_support/meshes/puzzle_piece/puzzle_bent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; visual mesh filename=package://tesseract_support/meshes/puzzle_piece/puzzle_bent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

File: tesseract_support/urdf/scene_graph_example.urdf (robot description, URDF)
Before this commit: robot irb2400_iiwa_cowork, 30 links, 29 joints
Links:
- link iiwa_base_link: geometry collision mesh filename=package://tesseract_support/meshes/lbr_iiwa_14_r820/collisi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; visual mesh filename=package://tesseract_support/meshes/lbr_iiwa_14_r820/visual/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
- link iiwa_link_1: geometry collision mesh filename=package://tesseract_support/meshes/lbr_iiwa_14_r820/collisi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; visual mesh filename=package://tesseract_support/meshes/lbr_iiwa_14_r820/visual/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
- link iiwa_link_2: geometry collision mesh filename=package://tesseract_support/meshes/lbr_iiwa_14_r820/collisi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; visual mesh filename=package://tesseract_support/meshes/lbr_iiwa_14_r820/visual/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
- link iiwa_link_3: geometry collision mesh filename=package://tesseract_support/meshes/lbr_iiwa_14_r820/collisi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; visual mesh filename=package://tesseract_support/meshes/lbr_iiwa_14_r820/visual/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
- link iiwa_link_4: geometry collision mesh filename=package://tesseract_support/meshes/lbr_iiwa_14_r820/collisi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; visual mesh filename=package://tesseract_support/meshes/lbr_iiwa_14_r820/visual/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
- link iiwa_link_5: geometry collision mesh filename=package://tesseract_support/meshes/lbr_iiwa_14_r820/collisi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; visual mesh filename=package://tesseract_support/meshes/lbr_iiwa_14_r820/visual/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
- link iiwa_link_6: geometry collision mesh filename=package://tesseract_support/meshes/lbr_iiwa_14_r820/collisi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; visual mesh filename=package://tesseract_support/meshes/lbr_iiwa_14_r820/visual/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
- link iiwa_link_7: geometry collision mesh filename=package://tesseract_support/meshes/lbr_iiwa_14_r820/collisi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; visual mesh filename=package://tesseract_support/meshes/lbr_iiwa_14_r820/visual/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
